Commit message: Add 20° nose-down pitch to D435 front camera URDF
The MakerWorld #1788451 D435 mount holds the camera angled nose-down
by design — the depth FOV covers the ground in front of the rig
instead of the horizon. Measured 2026-04-26 with a digital
inclinometer at ~20° (housing has a rounded top, ±2° uncertainty;
assumed the mount author used a round 20° rather than 23° or similar).

Without this rotation, RTABMap's depth fusion projects every point at
the wrong vertical position — at 3 m range, even 2° of unmodeled
pitch causes ~10 cm of vertical error. The 2D occupancy grid would
project distant floor as obstacles and break Nav2 costmap planning.

FAST-LIO2 is unaffected (it doesn't use the D435).

If the resulting RTABMap floor still looks tilted, the docs flag a
refinement procedure: fit a plane to depth points on a known-level
floor, take the angle between the plane normal and body +Z as the
residual pitch error.

Co-Authored-By: Claude Opus 4.7 (1M context) <noreply@anthropic.com>

File: urdf/sensors_common.urdf.xacro (robot description, xacro)
@@ -70,7 +70,17 @@
        realsense ROS macro applies internal optical offsets from
        this plane). Plate-Y -146.761 mm → body +X 146.761 mm.
-       Vertical center 28.502 mm below plate top. -->
+       Vertical center 28.502 mm below plate top.
+       Pitch: the MakerWorld #1788451 D435 mount has the camera
+       angled NOSE-DOWN by design (so the depth FOV covers the
+       ground in front of the rig, not the horizon). Measured with
+       a digital inclinometer on the rounded D435 housing top
+       (2026-04-26): ≈20°. Assumed exact 20° (round number per
+       mount author intent; housing rounded top gives ±2°
+       measurement uncertainty — refine with a depth-image
+       floor-plane fit if the map-tilt looks wrong in RTABMap).
+       REP-103: nose-down = NEGATIVE pitch.
+         20° × π/180 = 0.349066 rad → -0.349066 -->
   <xacro:property name="d435_front_xyz" value="0.146761 0.0 -0.028502"/>
-  <xacro:property name="d435_front_rpy" value="0.0 0.0 0.0"/>
+  <xacro:property name="d435_front_rpy" value="0.0 -0.349066 0.0"/>
   <!-- ============== Links + joints ============== -->
   <link name="sensor_plate">
