Commit message: Correct D435 front pitch to +10.09 deg (sign convention + measured value)
Two bugs in one fix.

(1) Sign convention. URDF rpy uses right-hand-rule rotation around +Y,
so positive pitch tilts +X (forward) toward -Z (down) -- ie POSITIVE
pitch = NOSE-DOWN. The previous comment claimed nose-down = NEGATIVE
pitch (aerospace convention) and stored -0.349 rad, which actually
encoded a 20 deg nose-UP rotation. The depth point cloud was
transformed accordingly and would have landed above the floor in any
gravity-anchored map.

(2) Wrong magnitude. The 20 deg nose-down value came from a digital
inclinometer reading on the rounded D435 housing top -- a surface
that is not perpendicular to the optical axis, so the reading was
unreliable. scripts/measure_d435_pitch.py with the rig on a level
floor (99.8% inlier fraction, 0.07 deg roll residual) measures the
actual pitch as +10.09 deg nose-down. Updating to 0.176136 rad.

After this fix re-running the script yields floor normal in base_link
= (+0.0002, -0.0012, +1.0000) and residual pitch error 0.01 deg --
confirming the corrected value.

File: urdf/sensors_common.urdf.xacro (robot description, xacro)
@@ -73,14 +73,20 @@
        Pitch: the MakerWorld #1788451 D435 mount has the camera
        angled NOSE-DOWN by design (so the depth FOV covers the
-       ground in front of the rig, not the horizon). Measured with
-       a digital inclinometer on the rounded D435 housing top
-       (2026-04-26): ≈20°. Assumed exact 20° (round number per
-       mount author intent; housing rounded top gives ±2°
-       measurement uncertainty — refine with a depth-image
-       floor-plane fit if the map-tilt looks wrong in RTABMap).
-       REP-103: nose-down = NEGATIVE pitch.
-         20° × π/180 = 0.349066 rad → -0.349066 -->
+       ground in front of the rig, not the horizon).
+       REP-103 / URDF rpy sign convention: pitch is right-hand
+       rotation around +Y (left), so R_y(+θ) takes +X (forward)
+       toward -Z (down). Therefore POSITIVE pitch = NOSE-DOWN.
+       (This is NOT aerospace convention — that one has +pitch =
+       nose-up. URDF rpy follows the right-hand-rule math.)
+       Measurement source (2026-04-26): scripts/measure_d435_pitch.py
+       with the rig on a level floor with clear FOV — 99.8% inlier
+       fraction on the floor plane fit, 0.07° roll residual (rig
+       confirmed level), reports actual pitch = +10.09° nose-down.
+       Inclinometer on the rounded D435 housing top earlier read
+       ~20°, but that surface is not perpendicular to the optical
+       axis and is unreliable. Trust the depth-plane fit.
+         10.09° × π/180 = 0.176136 rad -->
   <xacro:property name="d435_front_xyz" value="0.146761 0.0 -0.028502"/>
-  <xacro:property name="d435_front_rpy" value="0.0 -0.349066 0.0"/>
+  <xacro:property name="d435_front_rpy" value="0.0 0.176136 0.0"/>
   <!-- ============== Links + joints ============== -->
   <link name="sensor_plate">
