Commit message: fix: mecanum lidar height 0.108 → 0.292 m (tape-measured) + tilt-script floor selection
- mecanum.urdf.xacro: base_link_to_plate_top placeholder 0.107670 was
  18.4 cm short — plate top tape-measured at 11.5 in = 0.29210 m
  (2026-06-10). livox optical center now lands at 0.32871 m.
- slam.launch.py: PLATFORM_BRIDGES['mecanum'] z -0.144280 → -0.328710
  (plate_top + 0.03661 Livox offset), kept in lockstep per the comment.
- measure_lidar_tilt.py: select the LOWEST well-supported RANSAC plane
  instead of the most numerous — from a 0.33 m mount the floor is only
  visible past ~2.6 m at grazing angle and is outnumbered by furniture
  planes (the fit returned a couch 0.081 m below the sensor, refuted by
  tape measure). Range cap 6 → 10 m, and the report now cross-checks
  measured height against the URDF stack-up.

Co-Authored-By: Claude Fable 5 <noreply@anthropic.com>

File: urdf/mecanum.urdf.xacro (robot description, xacro)
@@ -6,13 +6,14 @@
   Stack-up (from base_link upward):
     base_link             Z = 0           (wheel contact / floor)
-        ↑ ~0.107670 m     chassis + sensor mast (UNMEASURED — placeholder)
-    sensor_plate          Z = 0.107670    (top of plate)
+        ↑ 0.29210 m       chassis + sensor mast (tape-measured 11.5 in,
+                          2026-06-10; replaces the old 0.107670
+                          placeholder that was off by 18.4 cm)
+    sensor_plate          Z = 0.29210     (top of plate)
         → see sensors_common.urdf.xacro for everything above this point
-  IMPORTANT: 0.107670 m is a PLACEHOLDER derived from slam.launch.py's
-  PLATFORM_BRIDGES mecanum entry (body → base_link = -0.144280 m) minus
-  the plate-top → livox_frame Z offset (36.61 mm per Livox datasheet).
-  Re-measure base_link → sensor-plate-top with calipers and update both
-  this xacro AND PLATFORM_BRIDGES['mecanum'] in slam.launch.py before
-  trusting the map z-axis.
+          (livox_frame optical center lands at 0.29210 + 0.03661
+           = 0.32871 m above the floor)
+  Kept in lockstep with PLATFORM_BRIDGES['mecanum'] in slam.launch.py
+  (body → base_link = -(plate_top + 0.03661) = -0.328710 m). If you
+  re-measure with calipers, update BOTH places.
   The chassis visual below is cosmetic only (RViz). Yahboom X3 outer
   dimensions are approximate; they don't affect SLAM math, only what
@@ -21,7 +22,7 @@
 <robot xmlns:xacro="http://www.ros.org/wiki/xacro" name="mecanum_x3">
   <xacro:include filename="$(find slam_bringup)/urdf/sensors_common.urdf.xacro"/>
-  <!-- Approximate Yahboom X3 chassis bbox — REPLACE with measured values
-       once a tape measure is in hand. -->
-  <xacro:property name="base_link_to_plate_top" value="0.107670"/>
+  <!-- Plate height tape-measured 11.5 in (2026-06-10). Chassis bbox below
+       is still approximate (cosmetic only). -->
+  <xacro:property name="base_link_to_plate_top" value="0.29210"/>
   <xacro:property name="chassis_length"         value="0.280"/>
   <xacro:property name="chassis_width"          value="0.230"/>
